Commit message: feat: update files

File: inspire_hand_left/urdf_left_with_force_sensor/urdf/urdf_left_with_force_sensor.urdf (robot description, URDF)
Before this commit: robot urdf_left_with_force_sensor, 30 links, 29 joints
Links:
- link base_link: geometry collision mesh filename=file:///Users/lr-2002/project/tele_hand/inspire_hand/inspir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; visual mesh filename=file:///Users/lr-2002/project/tele_hand/inspire_hand/inspir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
- link index_force_sensor_1: geometry collision mesh filename=file:///Users/lr-2002/project/tele_hand/inspire_hand/inspir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; visual mesh filename=file:///Users/lr-2002/project/tele_hand/inspire_hand/inspir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
- link index_force_sensor_2: geometry collision mesh filename=file:///Users/lr-2002/project/tele_hand/inspire_hand/inspir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; visual mesh filename=file:///Users/lr-2002/project/tele_hand/inspire_hand/inspir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
- link index_force_sensor_3: geometry collision mesh filename=file:///Users/lr-2002/project/tele_hand/inspire_hand/inspir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; visual mesh filename=file:///Users/lr-2002/project/tele_hand/inspire_hand/inspir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
- link left_index_1: geometry collision mesh filename=file:///Users/lr-2002/project/tele_hand/inspire_hand/inspir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; visual mesh filename=file:///Users/lr-2002/project/tele_hand/inspire_hand/inspir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
- link left_index_2: geometry collision mesh filename=file:///Users/lr-2002/project/tele_hand/inspire_hand/inspir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; visual mesh filename=file:///Users/lr-2002/project/tele_hand/inspire_hand/inspir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
- link left_little_1: geometry collision mesh filename=file:///Users/lr-2002/project/tele_hand/inspire_hand/inspir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; visual mesh filename=file:///Users/lr-2002/project/tele_hand/inspire_hand/inspir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
- link left_little_2: geometry collision mesh filename=file:///Users/lr-2002/project/tele_hand/inspire_hand/inspir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; visual mesh filename=file:///Users/lr-2002/project/tele_hand/inspire_hand/inspir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
- link left_middle_1: geometry collision mesh filename=file:///Users/lr-2002/project/tele_hand/inspire_hand/inspir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; visual mesh filename=file:///Users/lr-2002/project/tele_hand/inspire_hand/inspir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
- link left_middle_2: geometry collision mesh filename=file:///Users/lr-2002/project/tele_hand/inspire_hand/inspir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; visual mesh filename=file:///Users/lr-2002/project/tele_hand/inspire_hand/inspir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
- link left_ring_1: geometry collision mesh filename=file:///Users/lr-2002/project/tele_hand/inspire_hand/inspir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; visual mesh filename=file:///Users/lr-2002/project/tele_hand/inspire_hand/inspir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
- link left_ring_2: geometry collision mesh filename=file:///Users/lr-2002/project/tele_hand/inspire_hand/inspir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; visual mesh filename=file:///Users/lr-2002/project/tele_hand/inspire_hand/inspir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
- link left_thumb_1: geometry collision mesh filename=file:///Users/lr-2002/project/tele_hand/inspire_hand/inspir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; visual mesh filename=file:///Users/lr-2002/project/tele_hand/inspire_hand/inspir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
- link left_thumb_2: geometry collision mesh filename=file:///Users/lr-2002/project/tele_hand/inspire_hand/inspir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; visual mesh filename=file:///Users/lr-2002/project/tele_hand/inspire_hand/inspir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
- link left_thumb_3: geometry collision mesh filename=file:///Users/lr-2002/project/tele_hand/inspire_hand/inspir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; visual mesh filename=file:///Users/lr-2002/project/tele_hand/inspire_hand/inspir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
- link left_thumb_4: geometry collision mesh filename=file:///Users/lr-2002/project/tele_hand/inspire_hand/inspir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; visual mesh filename=file:///Users/lr-2002/project/tele_hand/inspire_hand/inspir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
- link little_force_sensor_1: geometry collision mesh filename=file:///Users/lr-2002/project/tele_hand/inspire_hand/inspir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; visual mesh filename=file:///Users/lr-2002/project/tele_hand/inspire_hand/inspir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
- link little_force_sensor_2: geometry collision mesh filename=file:///Users/lr-2002/project/tele_hand/inspire_hand/inspir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; visual mesh filename=file:///Users/lr-2002/project/tele_hand/inspire_hand/inspir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
- link little_force_sensor_3: geometry collision mesh filename=file:///Users/lr-2002/project/tele_hand/inspire_hand/inspir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; visual mesh filename=file:///Users/lr-2002/project/tele_hand/inspire_hand/inspir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
- link middle_force_sensor_1: geometry collision mesh filename=file:///Users/lr-2002/project/tele_hand/inspire_hand/inspir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; visual mesh filename=file:///Users/lr-2002/project/tele_hand/inspire_hand/inspir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
- link middle_force_sensor_2: geometry collision mesh filename=file:///Users/lr-2002/project/tele_hand/inspire_hand/inspir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; visual mesh filename=file:///Users/lr-2002/project/tele_hand/inspire_hand/inspir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
- link middle_force_sensor_3: geometry collision mesh filename=file:///Users/lr-2002/project/tele_hand/inspire_hand/inspir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; visual mesh filename=file:///Users/lr-2002/project/tele_hand/inspire_hand/inspir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
- link palm_force_sensor: geometry collision mesh filename=file:///Users/lr-2002/project/tele_hand/inspire_hand/inspir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; visual mesh filename=file:///Users/lr-2002/project/tele_hand/inspire_hand/inspir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
- link ring_force_sensor_1: geometry collision mesh filename=file:///Users/lr-2002/project/tele_hand/inspire_hand/inspir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; visual mesh filename=file:///Users/lr-2002/project/tele_hand/inspire_hand/inspir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
- link ring_force_sensor_2: geometry collision mesh filename=file:///Users/lr-2002/project/tele_hand/inspire_hand/inspir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; visual mesh filename=file:///Users/lr-2002/project/tele_hand/inspire_hand/inspir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
- link ring_force_sensor_3: geometry collision mesh filename=file:///Users/lr-2002/project/tele_hand/inspire_hand/inspir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; visual mesh filename=file:///Users/lr-2002/project/tele_hand/inspire_hand/inspir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
- link thumb_force_sensor_1: geometry collision mesh filename=file:///Users/lr-2002/project/tele_hand/inspire_hand/inspir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; visual mesh filename=file:///Users/lr-2002/project/tele_hand/inspire_hand/inspir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
- link thumb_force_sensor_2: geometry collision mesh filename=file:///Users/lr-2002/project/tele_hand/inspire_hand/inspir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; visual mesh filename=file:///Users/lr-2002/project/tele_hand/inspire_hand/inspir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
- link thumb_force_sensor_3: geometry collision mesh filename=file:///Users/lr-2002/project/tele_hand/inspire_hand/inspir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; visual mesh filename=file:///Users/lr-2002/project/tele_hand/inspire_hand/inspir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
- link thumb_force_sensor_4: geometry collision mesh filename=file:///Users/lr-2002/project/tele_hand/inspire_hand/inspir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; visual mesh filename=file:///Users/lr-2002/project/tele_hand/inspire_hand/inspir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
